File: RF_ProtoBoard_Extended/RF_ProtoBoard_Extended.kicad_sch (KiCad schematic)
At the start: 12 parts, among them J1 Screw_Terminal_01x02, J2 Conn_VPlus_Gnd

Commit message: Excluded from BOM, disable allow_soldermask_bridges
Parts:
- A1, A2, A3, A4, A5, A6, J2: now left out of the parts list
Changed lines of the file:
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@@
   )
   (symbol (lib_id "RF_ProtoBoard:Conn_VPlus_Gnd") (at 53.975 363.22 270) (unit 1)
-    (in_bom yes) (on_board yes) (dnp no)
+    (in_bom no) (on_board yes) (dnp no)
     (property "Reference" "J2" (at 48.895 361.95 90)
       (effects (font (size 1.27 1.27)) (justify right))
@@
   )
   (symbol (lib_id "RF_ProtoBoard:GndRing_RF_ProtoBoard_Module") (at 146.685 270.51 0) (unit 1)
-    (in_bom yes) (on_board yes) (dnp no)
+    (in_bom no) (on_board yes) (dnp no)
     (property "Reference" "A5" (at 146.685 253.365 0)
       (effects (font (size 1.27 1.27)))
@@
   )
   (symbol (lib_id "RF_ProtoBoard:GndRing_RF_ProtoBoard_Module") (at 146.685 166.37 0) (unit 1)
-    (in_bom yes) (on_board yes) (dnp no)
+    (in_bom no) (on_board yes) (dnp no)
     (property "Reference" "A3" (at 146.685 149.225 0)
       (effects (font (size 1.27 1.27)))
@@
   )
   (symbol (lib_id "RF_ProtoBoard:GndRing_RF_ProtoBoard_Module") (at 146.685 114.3 0) (unit 1)
-    (in_bom yes) (on_board yes) (dnp no)
+    (in_bom no) (on_board yes) (dnp no)
     (property "Reference" "A2" (at 146.685 97.155 0)
       (effects (font (size 1.27 1.27)))
@@
   )
   (symbol (lib_id "RF_ProtoBoard:GndRing_RF_ProtoBoard_Module") (at 146.685 219.075 0) (unit 1)
-    (in_bom yes) (on_board yes) (dnp no)
+    (in_bom no) (on_board yes) (dnp no)
     (property "Reference" "A4" (at 146.685 201.93 0)
       (effects (font (size 1.27 1.27)))
@@
   )
   (symbol (lib_id "RF_ProtoBoard:GndRing_RF_ProtoBoard_Module") (at 146.685 322.58 0) (unit 1)
-    (in_bom yes) (on_board yes) (dnp no)
+    (in_bom no) (on_board yes) (dnp no)
     (property "Reference" "A6" (at 146.685 305.435 0)
       (effects (font (size 1.27 1.27)))
@@
   )
   (symbol (lib_id "RF_ProtoBoard:GndRing_RF_ProtoBoard_Module") (at 146.685 62.865 0) (unit 1)
-    (in_bom yes) (on_board yes) (dnp no)
+    (in_bom no) (on_board yes) (dnp no)
     (property "Reference" "A1" (at 146.685 45.72 0)
       (effects (font (size 1.27 1.27)))
