File: RF_ProtoBoard_Extended/RF_ProtoBoard_Extended.kicad_pcb (KiCad board)
At the start: 2 copper layers, 99.6 x 87.6 mm, 12 parts, among them J1 Screw_Terminal_01x02, J2 Conn_VPlus_Gnd

Commit message: Excluded from BOM, disable allow_soldermask_bridges
Parts:
- A1, A2, A3, A4, A5, A6: value (none) -> GndRing_RF_ProtoBoard_Module
Changed lines of the file:
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@@
     (property "ki_description" "Mounting Hole without connection")
     (property "ki_keywords" "mounting hole")
-    (attr exclude_from_pos_files exclude_from_bom)
+    (attr exclude_from_pos_files)
     (fp_text reference "H3" (at 0 -3.7) (layer "F.SilkS") hide
         (effects (font (size 1 1) (thickness 0.15)))
@@
     (property "Sheetfile" "RF_ProtoBoard_Extended.kicad_sch")
     (property "Sheetname" "")
+    (property "exclude_from_bom" "")
     (property "ki_keywords" "RF Radio Frequency Connector Protoboard")
-    (attr allow_soldermask_bridges)
+    (attr exclude_from_bom allow_soldermask_bridges)
     (fp_text reference "A4" (at 0 17.78 unlocked) (layer "F.SilkS") hide
         (effects (font (size 1 1) (thickness 0.15)))
     )
-    (fp_text value " " (at 0 -17.78) (layer "F.Fab") hide
+    (fp_text value "GndRing_RF_ProtoBoard_Module" (at 0 -17.78) (layer "F.Fab") hide
         (effects (font (size 1 1) (thickness 0.15)))
     )
@@
     (property "ki_description" "Mounting Hole without connection")
     (property "ki_keywords" "mounting hole")
-    (attr exclude_from_pos_files exclude_from_bom)
+    (attr exclude_from_pos_files)
     (fp_text reference "H2" (at 0 -3.7) (layer "F.SilkS") hide
         (effects (font (size 1 1) (thickness 0.15)))
@@
     (property "Sheetfile" "RF_ProtoBoard_Extended.kicad_sch")
     (property "Sheetname" "")
+    (property "exclude_from_bom" "")
     (property "ki_keywords" "RF Radio Frequency Connector Protoboard")
-    (attr allow_soldermask_bridges)
+    (attr exclude_from_bom allow_soldermask_bridges)
     (fp_text reference "A1" (at 0 17.78 unlocked) (layer "F.SilkS") hide
         (effects (font (size 1 1) (thickness 0.15)))
     )
-    (fp_text value " " (at 0 -17.78) (layer "F.Fab") hide
+    (fp_text value "GndRing_RF_ProtoBoard_Module" (at 0 -17.78) (layer "F.Fab") hide
         (effects (font (size 1 1) (thickness 0.15)))
     )
@@
     (property "ki_description" "Mounting Hole without connection")
     (property "ki_keywords" "mounting hole")
-    (attr exclude_from_pos_files exclude_from_bom)
+    (attr exclude_from_pos_files)
     (fp_text reference "H4" (at 0 -3.7) (layer "F.SilkS") hide
         (effects (font (size 1 1) (thickness 0.15)))
@@
     (property "Sheetfile" "RF_ProtoBoard_Extended.kicad_sch")
     (property "Sheetname" "")
+    (property "exclude_from_bom" "")
     (property "ki_keywords" "RF Radio Frequency Connector Protoboard")
-    (attr allow_soldermask_bridges)
+    (attr exclude_from_bom allow_soldermask_bridges)
     (fp_text reference "A2" (at 0 17.78 unlocked) (layer "F.SilkS") hide
         (effects (font (size 1 1) (thickness 0.15)))
     )
-    (fp_text value " " (at 0 -17.78) (layer "F.Fab") hide
+    (fp_text value "GndRing_RF_ProtoBoard_Module" (at 0 -17.78) (layer "F.Fab") hide
         (effects (font (size 1 1) (thickness 0.15)))
     )
@@
     (property "Sheetfile" "RF_ProtoBoard_Extended.kicad_sch")
     (property "Sheetname" "")
+    (property "exclude_from_bom" "")
     (property "ki_keywords" "RF Radio Frequency Connector Protoboard")
-    (attr allow_soldermask_bridges)
+    (attr exclude_from_bom allow_soldermask_bridges)
     (fp_text reference "A3" (at 0 17.78 unlocked) (layer "F.SilkS") hide
         (effects (font (size 1 1) (thickness 0.15)))
     )
-    (fp_text value " " (at 0 -17.78) (layer "F.Fab") hide
+    (fp_text value "GndRing_RF_ProtoBoard_Module" (at 0 -17.78) (layer "F.Fab") hide
         (effects (font (size 1 1) (thickness 0.15)))
     )
@@
     (property "Sheetfile" "RF_ProtoBoard_Extended.kicad_sch")
     (property "Sheetname" "")
+    (property "exclude_from_bom" "")
     (property "ki_keywords" "RF Radio Frequency Connector Protoboard")
-    (attr allow_soldermask_bridges)
+    (attr exclude_from_bom allow_soldermask_bridges)
     (fp_text reference "A6" (at 0 17.78 unlocked) (layer "F.SilkS") hide
         (effects (font (size 1 1) (thickness 0.15)))
     )
-    (fp_text value " " (at 0 -17.78) (layer "F.Fab") hide
+    (fp_text value "GndRing_RF_ProtoBoard_Module" (at 0 -17.78) (layer "F.Fab") hide
         (effects (font (size 1 1) (thickness 0.15)))
     )
@@
     (property "ki_description" "Mounting Hole without connection")
     (property "ki_keywords" "mounting hole")
-    (attr exclude_from_pos_files exclude_from_bom)
+    (attr exclude_from_pos_files)
     (fp_text reference "H1" (at 0 -3.7) (layer "F.SilkS") hide
         (effects (font (size 1 1) (thickness 0.15)))
@@
     (property "Sheetfile" "RF_ProtoBoard_Extended.kicad_sch")
     (property "Sheetname" "")
+    (property "exclude_from_bom" "")
     (property "ki_keywords" "RF Radio Frequency Connector Protoboard")
-    (attr allow_soldermask_bridges)
+    (attr exclude_from_bom allow_soldermask_bridges)
     (fp_text reference "A5" (at 0 17.78 unlocked) (layer "F.SilkS") hide
         (effects (font (size 1 1) (thickness 0.15)))
     )
-    (fp_text value " " (at 0 -17.78) (layer "F.Fab") hide
+    (fp_text value "GndRing_RF_ProtoBoard_Module" (at 0 -17.78) (layer "F.Fab") hide
         (effects (font (size 1 1) (thickness 0.15)))
     )
@@
     (property "Sheetfile" "RF_ProtoBoard_Extended.kicad_sch")
     (property "Sheetname" "")
+    (property "exclude_from_bom" "")
     (property "ki_description" "Power connector, single row, 01x02, power distribution")
     (property "ki_keywords" "power connector")
-    (attr through_hole)
+    (attr through_hole exclude_from_bom)
     (fp_text reference "J2" (at 0 3.302 unlocked) (layer "F.SilkS") hide
         (effects (font (size 1 1) (thickness 0.1)))

Commit message: Excluded from BOM, disable allow_soldermask_bridges
Parts:
- A1, A2, A3, A4, A5, A6: value GndRing_RF_ProtoBoard_Module -> (none)
