File: RF_ProtoBoard_Extended/RF_ProtoBoard_Extended.kicad_pcb (KiCad board)
At the start: 2 copper layers, 99.6 x 87.6 mm, 12 parts, among them J1 Screw_Terminal_01x02, J2 Conn_VPlus_Gnd

Commit message: add "JLCJLCJLCJLC" to back silkscreen layer, to specify location of  JLCPCB order number
Other:
- board text added: "JLCJLCJLCJLC"
Changed lines of the file:
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@@
   (gr_rect (start 17.78 17.78) (end 114.3 81.28)
     (stroke (width 0.1) (type default)) (fill none) (layer "User.1"))
+  (gr_text "JLCJLCJLCJLC" (at 66.04 86.36) (layer "B.SilkS")
+    (effects (font (size 1 1) (thickness 0.15)) (justify bottom mirror))
+  )
   (segment (start 68.54 13.462) (end 68.54 6.35) (width 2.4) (layer "F.Cu") (net 721))
   (segment (start 63.54 13.462) (end 63.54 6.35) (width 2.4) (layer "F.Cu") (net 722))
