File: RF_ProtoBoard_Extended/RF_ProtoBoard_Extended.kicad_pcb (KiCad board)
At the start: 2 copper layers, 99.6 x 87.6 mm, 12 parts, among them J1 Screw_Terminal_01x02, J2 Conn_VPlus_Gnd

Commit message: Add version number to the backside silkscreen
Other:
- board text added: "Version 1.0"
Changed lines of the file:
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@@
   (gr_rect (start 17.78 17.78) (end 114.3 81.28)
     (stroke (width 0.1) (type default)) (fill none) (layer "User.1"))
-  (gr_text "JLCJLCJLCJLC" (at 66.04 86.36) (layer "B.SilkS")
+  (gr_text "JLCJLCJLCJLC" (at 66.04 86.106) (layer "B.SilkS")
     (effects (font (size 1 1) (thickness 0.15)) (justify bottom mirror))
   )
+  (gr_text "Version 1.0" (at 66.04 87.884) (layer "B.SilkS")
+    (effects (font (size 1 1) (thickness 0.15)) (justify bottom mirror))
+  )

Commit message: Set PCB's revision variable, and automatically update back silkscreen accordingly
Other:
- board text added: "${REVISION}"
- board text removed: "Version 1.0"
Changed lines of the file:
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@@
   )
   (paper "A4")
+  (title_block
+    (date "2023-09-19")
+    (rev "Version 1.0")
+  )
   (layers
     (0 "F.Cu" signal)
@@
     (effects (font (size 1 1) (thickness 0.15)) (justify bottom mirror))
   )
-  (gr_text "Version 1.0" (at 66.04 87.884) (layer "B.SilkS")
+  (gr_text "${REVISION}" (at 66.04 87.884) (layer "B.SilkS")
     (effects (font (size 1 1) (thickness 0.15)) (justify bottom mirror))
   )

Commit message: Add ProductNumberPlaceholder text variable; makes it easier to change placeholder text (or entirely remove it) depending on manufacturer
Other:
- board text added: "${ProductNumberPlaceholder}"
- board text removed: "JLCJLCJLCJLC"
Changed lines of the file:
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@@
     )
   )
+  (property "ProductNumberPlaceholder" "JLCJLCJLCJLC")
   (net 0 "")
   (net 1 "GND1")
@@
   (gr_rect (start 17.78 17.78) (end 114.3 81.28)
     (stroke (width 0.1) (type default)) (fill none) (layer "User.1"))
-  (gr_text "JLCJLCJLCJLC" (at 66.04 86.106) (layer "B.SilkS")
+  (gr_text "${ProductNumberPlaceholder}" (at 66.04 86.106) (layer "B.SilkS")
     (effects (font (size 1 1) (thickness 0.15)) (justify bottom mirror))
   )
