File: RF_ProtoBoard/RF_ProtoBoard.kicad_pcb (KiCad board)
At the start: 2 copper layers, 96.5 x 63.5 mm, 6 parts

Commit message: Fix courtyard and solder_mask_bridges warning
Parts:
- A1, A2, A3, A4, A5, A6: value RF_ProtoBoard_Module -> (none)

Commit message: -
Parts:
- A1, A2, A3, A4, A5, A6: value (none) -> RF_ProtoBoard_Module
Changed lines of the file:
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@@
         (effects (font (size 1 1) (thickness 0.15)))
     )
-    (fp_text value " " (at 0 -17.78) (layer "F.Fab") hide
+    (fp_text value "RF_ProtoBoard_Module" (at 0 -17.78) (layer "F.Fab") hide
         (effects (font (size 1 1) (thickness 0.15)))
     )
@@
         (effects (font (size 1 1) (thickness 0.15)))
     )
-    (fp_text value " " (at 0 -17.78) (layer "F.Fab") hide
+    (fp_text value "RF_ProtoBoard_Module" (at 0 -17.78) (layer "F.Fab") hide
         (effects (font (size 1 1) (thickness 0.15)))
     )
@@
         (effects (font (size 1 1) (thickness 0.15)))
     )
-    (fp_text value " " (at 0 -17.78) (layer "F.Fab") hide
+    (fp_text value "RF_ProtoBoard_Module" (at 0 -17.78) (layer "F.Fab") hide
         (effects (font (size 1 1) (thickness 0.15)))
     )
@@
         (effects (font (size 1 1) (thickness 0.15)))
     )
-    (fp_text value " " (at 0 -17.78) (layer "F.Fab") hide
+    (fp_text value "RF_ProtoBoard_Module" (at 0 -17.78) (layer "F.Fab") hide
         (effects (font (size 1 1) (thickness 0.15)))
     )
@@
         (effects (font (size 1 1) (thickness 0.15)))
     )
-    (fp_text value " " (at 0 -17.78) (layer "F.Fab") hide
+    (fp_text value "RF_ProtoBoard_Module" (at 0 -17.78) (layer "F.Fab") hide
         (effects (font (size 1 1) (thickness 0.15)))
     )
@@
         (effects (font (size 1 1) (thickness 0.15)))
     )
-    (fp_text value " " (at 0 -17.78) (layer "F.Fab") hide
+    (fp_text value "RF_ProtoBoard_Module" (at 0 -17.78) (layer "F.Fab") hide
         (effects (font (size 1 1) (thickness 0.15)))
     )

Commit message: exclude from bom and pos files
Parts:
- A1, A2, A3, A4, A5, A6: value RF_ProtoBoard_Module -> (none)
