File: RF_ProtoBoard/RF_ProtoBoard.kicad_pcb (KiCad board)
At the start: 2 copper layers, 96.5 x 63.5 mm, 6 parts

Commit message: add "JLCJLCJLCJLC" to back silkscreen layer, to specify location of  JLCPCB order number
Other:
- board text added: "JLCJLCJLCJLC"
Changed lines of the file:
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@@
   (gr_rect (start 17.78 17.78) (end 114.3 81.28)
     (stroke (width 0.1) (type default)) (fill none) (layer "Edge.Cuts"))
+  (gr_text "JLCJLCJLCJLC" (at 113.411 50.165) (layer "B.SilkS")
+    (effects (font (size 1 1) (thickness 0.15)) (justify left bottom mirror))
+  )
   (zone (net 601) (net_name "GND6") (layer "B.Cu") (hatch edge 0.5)
     (priority 5)
